Commit message: 更新readme

File: src/my_robot_description/urdf/robot.urdf (robot description, URDF)
Before this commit: robot my_car, 2 links, 1 joints
Links:
- added link left_wheel; visual cylinder length=0.03 radius=0.06
- added link right_wheel; visual cylinder length=0.03 radius=0.06
- link base_link: geometry visual box size=0.40 0.30 0.10
Joints:
- added joint left_wheel_joint: type continuous, parent base_link, child left_wheel, origin xyz=0 0.165 0 rpy=0 0 0, axis 0 1 0
- added joint right_wheel_joint: type continuous, parent base_link, child right_wheel, origin xyz=0 -0.165 0 rpy=0 0 0, axis 0 1 0
- joint base_footprint_joint: origin xyz=0 0 0.05 rpy=0 0 0 -> xyz=0 0 0.06 rpy=0 0 0

Commit message: Gazebo 仿真：URDF 物理属性、差速驱动、看门狗、雷达、相机 + cv_bridge
新增文件：
- my_robot_description/launch/gazebo.launch.py      启动 Gazebo + 生成模型 + 看门狗
- my_robot_description/worlds/my_world.world        仿真场景（地面 + 方块/圆柱/墙）
- my_first_pkg/src/cmd_vel_watchdog.cpp             速度指令看门狗（超时自动停车）
- my_first_pkg/src/image_processor.cpp              cv_bridge + OpenCV 边缘检测
- my_first_pkg/config/image_processor.yaml          参数持久化
- my_first_pkg/launch/image_processor.launch.py     带参数文件的启动

修改文件：
- urdf/robot.urdf           补 inertial/collision、前后万向轮、激光雷达、相机、差速驱动插件
- my_first_pkg/CMakeLists.txt、package.xml          新增两个节点与 sensor_msgs/cv_bridge 依赖
- my_robot_description/CMakeLists.txt               安装 worlds 目录
- README.md                 新增 12~15 节、Gazebo 运行方式、Demo 一览补 2 项、开发记录（按日期）

File: src/my_robot_description/urdf/robot.urdf (robot description, URDF)
Before this commit: robot my_car, 4 links, 3 joints
Links:
- added link camera_link, mass 0.05; collision box size=0.03 0.03 0.03; visual box size=0.03 0.03 0.03
- added link caster_front, mass 0.1; collision sphere radius=0.03; visual sphere radius=0.03
- added link caster_rear, mass 0.1; collision sphere radius=0.03; visual sphere radius=0.03
- added link lidar_link, mass 0.1; collision cylinder length=0.04 radius=0.035; visual cylinder length=0.04 radius=0.035
- link base_link: mass None -> 2.0; geometry collision box size=0.40 0.30 0.10; visual box size=0.40 0.30 0.10
- link left_wheel: mass None -> 0.3; geometry collision cylinder length=0.03 radius=0.06; visual cylinder length=0.03 radius=0.06
- link right_wheel: mass None -> 0.3; geometry collision cylinder length=0.03 radius=0.06; visual cylinder length=0.03 radius=0.06
Joints:
- added joint camera_joint: type fixed, parent base_link, child camera_link, origin xyz=0.22 0 0.02 rpy=0 0 0
- added joint caster_front_joint: type fixed, parent base_link, child caster_front, origin xyz=0.15 0 -0.03 rpy=0 0 0
- added joint caster_rear_joint: type fixed, parent base_link, child caster_rear, origin xyz=-0.15 0 -0.03 rpy=0 0 0
- added joint lidar_joint: type fixed, parent base_link, child lidar_link, origin xyz=0 0 0.07 rpy=0 0 0
- joint left_wheel_joint: limit (none) -> effort=10 velocity=30
- joint right_wheel_joint: limit (none) -> effort=10 velocity=30
